File: pi-top_Template.sch (KiCad schematic (older format))
At the start: 2 parts, among them J1 CONN_02X17, J2 CONN_02X17

Commit message: Shuffling files around for a "standard" workspace
Parts:
- J1: footprint library:Harwin_M22-5431705 -> pi-top:3M_951217-4620-XX
- J2: footprint library:Harwin_M22-6553442R -> pi-top:Harwin_M22-6553442R
Changed lines of the file:
@@
 LIBS:contrib
 LIBS:valves
-LIBS:pi-topT-Proto-cache
 EELAYER 26 0
 EELAYER END
@@
 F 0 "J1" H 3350 5015 50  0000 C CNN
 F 1 "CONN_02X17" H 3350 4924 50  0000 C CNN
-F 2 "library:Harwin_M22-5431705" H 3350 2900 50  0001 C CNN
+F 2 "pi-top:3M_951217-4620-XX" H 3350 2900 50  0001 C CNN
 F 3 "" H 3350 2900 50  0001 C CNN
 	1    3350 4000
@@
 F 0 "J2" H 7950 5015 50  0000 C CNN
 F 1 "CONN_02X17" H 7950 4924 50  0000 C CNN
-F 2 "library:Harwin_M22-6553442R" H 7950 2900 50  0001 C CNN
+F 2 "pi-top:Harwin_M22-6553442R" H 7950 2900 50  0001 C CNN
 F 3 "" H 7950 2900 50  0001 C CNN
 	1    7950 4000
